File: PCB/Lattice PCB/FPGA_DENDY_LAT.sch (EAGLE design)
At the start: 165 parts, among them CN1 DENDY60PINSLOT, J9 BYPASS, U1 LCMXO2-4000HC-4TG144C, U10 THS7374IPWR, U11 SN74LVC1G125DBVR, U12 SN74LVC1G240DBVR, U13 SN74LVC1G240DBVR, U14 SN74LVC1G240DBVR, U15 SN74LVC1G240DBVR, U16 OPA2134U, U2 74LS373WMSO20, U3 SN74LVC8T245, U4 SN74LVCH16T245DGGR, U5 SN74LVCH16T245DGGR, U6 74LVC1G04GV, U7 SN74LVC2G04DBVR, U8 SN74LVC2G34DBVR, U9 SN74LVC2G34DBVR, X1 057-010-1, X2 JOYPAD1, X3 9V, X4 JOYPAD2

Commit message: Add files via upload
Parts:
- U3: device SnapEDA-Library:SN74LVC8T245 -> SN74LVC8T245:SN74LVC8T245
Other:
- moved on the sheet: C14, C15, C2, C3, R2, R3, U6, U7, U8, U9
