File: PCB/Cyclone PCB/FPGA_DENDY.sch (EAGLE design)
At the start: 172 parts, among them CN1 DENDY60PINSLOT, J9 BYPASS, U1 EP2C5T144, U10 SN74LVC2G34DBVR, U11 THS7374IPWR, U12 SN74LVC1G125DBVR, U13 SN74LVC1G240DBVR, U14 SN74LVC1G240DBVR, U15 SN74LVC1G240DBVR, U16 SN74LVC1G240DBVR, U17 OPA2134U, U2 74LS373WMSO20, U3 SN74LVC8T245, U4 SN74LVCH16T245DGGR, U5 SN74LVCH16T245DGGR, U6 74LVC1G04GV, U7 EPCS4, U8 SN74LVC2G04DBVR, U9 SN74LVC2G34DBVR, X1 057-010-1, X2 JOYPAD1, X3 9V, X4 JOYPAD2

Commit message: Add files via upload
Parts:
- added C62: 10uF, rcl_my:CPOL-EU153CLV-0505
- added C63: 0.1uF, rcl_my:C-EUC0805
- added C64: 10uF, rcl_my:C-EUC0805
- added LED2: GNL-1206YC, led:LEDSML1206
- added R58: 1.2k, rcl:R-EU_R0805
- added R59, R60, R61, R62: 10k, rcl:R-EU_R0805
- C19, C26, C27: value 1uF -> 0.1uF
- C21, C34, C35: value 0.1uF -> 1uF
- C23: value 0.1uF -> 1000
- C25, C30: value 0.1uF -> 10uF; device rcl_my:C-EUC0805 -> rcl_my:CPOL-EU153CLV-0505
- C29: value 100uF -> 0.1uF; device rcl_my:CPOL-EU153CLV-0505 -> rcl_my:C-EUC0805
- C32: value 100uF -> 1000; device rcl_my:CPOL-EU153CLV-0505 -> rcl_my:C-EUC0805
- C37: value 22uF -> 100uF
- C39, C42, C47: value 1000 -> 0.1uF
- C40: value 10uF -> 100uF
- C43: value 10uF -> 0.1uF; device rcl_my:CPOL-EU153CLV-0505 -> rcl_my:C-EUC0805
- C45: value 1000 -> 22uF; device rcl_my:C-EUC0805 -> rcl_my:CPOL-EU153CLV-0505
- C49: value 0.01uF -> 0.1uF
- C50: value 0.1uF -> 1000; device rcl_my:C-EUC0603 -> rcl_my:C-EUC0805
- C51: value 22uF -> 1000; device rcl_my:C-EUC0603 -> rcl_my:C-EUC0805
- C52: value 0.1uF -> 0.01uF; device rcl_my:C-EUC0603 -> rcl_my:C-EUC0805
- C53: device rcl_my:C-EUC0805 -> rcl_my:C-EUC0603
- C54: value 0.1uF -> 22uF; device rcl_my:C-EUC0805 -> rcl_my:C-EUC0603
- C55: value 10uF -> 0.1uF; device rcl_my:C-EUC0805 -> rcl_my:C-EUC0603
- C56: value 10uF -> 0.1uF
- C58, C59: device rcl_my:CPOL-EU153CLV-0505 -> rcl_my:C-EUC0805
- C61: device rcl_my:C-EUC0805 -> rcl_my:CPOL-EU153CLV-0505
- U3: device SnapEDA-Library:SN74LVC8T245 -> SN74LVC8T245:SN74LVC8T245
Connections:
- removed net PD_DIR: U1.IO16, U3.DIR
- new net 6502_T1: R58.2, U1.IO16
- new net N$3: LED2.A, R58.1
- net +5V: now also C39.1, C40.+, C41.1, C53.2, C54.2, C55.2, C56.1, C57.1, U3.VCCA; no longer C31.1, C32.+, C33.1, C50.2, C51.2, C52.2, C53.1, C54.1, U3.VCCB@1, U3.VCCB@2
- net /IN0: now also R60.2
- net /IN1: now also R59.2
- net /PRD_FPGA: now also R61.1, U3.DIR
- net /RESET: now also C18.2; no longer C17.2
- net DB_DIR: now also R62.2
- net DMC: now also C52.2; no longer C49.2
- net GND: now also C17.2, C22.1, C23.1, C24.1, C25.-, C26.1, C29.2, C30.-, C32.2, C43.2, C45.-, C48.2, C49.2, C50.2, C53.1, C54.1, C55.1, C56.2, C57.2, C60.1, C63.2, C64.2, LED2.C, R61.2; no longer C17.1, C22.2, C23.2, C24.2, C25.2, C26.2, C29.-, C30.2, C32.-, C43.-, C45.2, C48.1, C49.1, C50.1, C53.2, C54.2, C57.1, C60.2, C61.2
- net LCH: now also C62.-; no longer C59.-
- net N$1: now also C58.1; no longer C55.1
- net N$30: now also C59.1; no longer C56.1
- net N$37: now also C61.+; no longer C58.+
- net N$4: now also C58.2; no longer C55.2
- net N$5: now also C59.2; no longer C56.2
- net N$7: now also C62.+; no longer C59.+
- net RCH: now also C61.-; no longer C58.-
- net SND_DAC: now also C51.2; no longer C48.2
- net VAPLL1: now also C30.+, C31.1, C32.1, L2.2; no longer C38.1, C39.1, C40.+, L1.2
- net VAPLL2: now also C23.2, C24.2, C25.+, L1.1; no longer C41.1, C42.1, C43.+, L2.2
- net VCC: now also C37.+, C38.1, C60.2; no longer C29.+, C30.1, C57.2
- net VCCINT: now also C17.1, C21.2, C26.2, C34.1, C35.1, C44.1, C45.+, L1.2; no longer C19.2, C26.1, C27.1, C36.1, C37.+, L1.1
- net VCCIO: now also C19.2, C22.2, C27.1, C29.1, C33.1, C36.1, C42.1, C43.1, C48.1, C49.1, C50.1, R59.1, R60.1, R62.1, U3.VCCB@1, U3.VCCB@2; no longer C18.2, C21.2, C22.1, C23.1, C24.1, C25.1, C34.1, C35.1, C44.1, C45.1, U3.VCCA
- net VPPL3: now also C63.1, C64.1; no longer C60.1, C61.1
Other:
- note added: "6502 T1"
- moved on the sheet: C14, C15, C16, C17, C18, C19, C2, C20, C21, C22, C23, C24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

Commit message: Add files via upload
Parts:
- removed R59, R60, R61, R62: 10k, rcl:R-EU_R0805
- added D3: 1N4148, diode:DIODE-DO214AA
- added RN15: 4k7, resistor-dil:4R-N0603-ARC
- R1: value 4k7 -> 1.2k
- R10, R9: value 51 -> 10k
- R11: value 2k -> 10k
- R12, R14, RN14: value 4k7 -> 10k
- R13, R45: value 4k7 -> 1k
- R15: value 287 -> 51
- R16: value 750 -> 51
- R17: value 124 -> 4k7
- R18: value 287 -> 4k7
- R19: value 750 -> 4k7
- R2, R44: value 1k -> 2k
- R20, R23: value 124 -> 287
- R21: value 287 -> 750
- R22: value 750 -> 124
- R24: value 2k -> 750
- R25, R28: value 2k -> 124
- R26: value 2k -> 287
- R27: value 1k -> 750
- R29: value 820 -> 2k
- R3: value 1k -> 4k7
- R31: value 10 -> 2k
- R32: value 1,1k -> 1k
- R33: value 510 -> 2k
- R34: value 4.7k -> 820
- R35: value 75 -> 2k
- R36: value 75 -> 10
- R37: value 75 -> 1,1k
- R38: value 75 -> 510
- R39: value 10k -> 4.7k
- R40, R41, R42: value 10k -> 75
- R43: value 2k -> 75
- R46: value 2k2 -> 4k7
- R47: value 4k7 -> 2k2
- R48: value 2k -> 4k7
- R49: value 1k5 -> 2k
- R50: value 1k -> 1k5
- R51, R56, R7: value 10k -> 1k
- R52, R57: value 10 -> 10k
- R53: value 1k -> 10
- R58: value 1.2k -> 10
Connections:
- removed net N$64: R35.1, U11.CH1_OUT
- removed net N$65: R36.1, U11.CH2_OUT
- removed net N$66: R37.1, U11.CH3_OUT
- removed net N$67: R38.1, U11.CH4_OUT
- new net N$15: R43.1, U11.CH4_OUT
- new net N$20: R42.1, U11.CH3_OUT
- new net N$21: R41.1, U11.CH2_OUT
- new net N$22: R40.1, U11.CH1_OUT
- new net N$46: D3.C, X1-4.S
- net #CS: now also R43.2; no longer R38.2
- net +5V: now also R3.1, R36.1, RN14A.1, RN14B.2, RN14C.2, RN14D.2; no longer R1.1, R31.1, R34.1, R40.1, R41.1, R42.1
- net /DENDY: now also R18.2; no longer R13.2
- net /IN0: now also R5.2; no longer R60.2
- net /IN1: now also R6.2; no longer R59.2
- net /IRQ: now also R3.2; no longer R1.2
- net /PAL: now also R17.2; no longer R12.2
- net /PRD_FPGA: now also R14.1; no longer R61.1
- net /RESET: now also R19.2; no longer R14.2
- net 6502_T1: now also R1.2; no longer R58.2
- net B: now also R40.2; no longer R35.2
- net CLKN: now also R15.2; no longer R9.2
- net CLKP: now also R16.2; no longer R10.2
- net CONF_DONE: now also R9.2; no longer R4.2
- net CS_FPGA: now also R37.2; no longer R32.2
- net DB_DIR: now also R4.2; no longer R62.2
- net DMC: now also R34.2, R35.1, R45.1, R49.1; no longer R29.2, R30.1, R44.1, R48.1
- net DMC_PWM: now also R34.1; no longer R29.1
- net EMPH_B: now also R21.1; no longer R16.1
- net EMPH_G: now also R24.1; no longer R19.1
- net EMPH_R: now also R27.1; no longer R22.1
- net G: now also R41.2; no longer R36.2
- net GND: now also R12.2, R13.2, R14.2, R20.1, R23.1, R26.1, R29.2, R35.2, R38.1, R47.2, R55.2, RN15A.1, RN15D.1; no longer R15.1, R18.1, R21.1, R24.2, R28.1, R30.2, R46.2, R54.2, R61.2, R7.2, R8.2, RN14A.1, RN14D.1
- net JOYDATA1: now also RN14D.1; no longer R39.2
- net JOYDATA2: now also RN14C.1; no longer R41.2
- net N$1: now also R46.2; no longer R43.2
- net N$14: now also R21.2, R22.1; no longer R16.2, R17.1
- net N$19: now also R31.2, R32.1; no longer R26.2, R27.1
- net N$2: now also R16.1; no longer R10.1
- net N$24: now also R24.2, R25.1; no longer R19.2, R20.1
- net N$3: now also LED1.A, R1.1; no longer LED2.A, R58.1
- net N$30: now also R50.2; no longer R47.2
- net N$34: now also R27.2, R28.1; no longer R22.2, R23.1
- net N$37: now also R53.2; no longer R52.2
- net N$38: now also R23.2, R25.2; no longer R18.2, R20.2
- net N$4: now also RN15C.1, RN15D.2; no longer RN14C.1, RN14D.2
- net N$42: now also R51.2, R52.1; no longer R50.2, R51.1
- net N$43: now also R52.2, R53.1; no longer R51.2, R52.1
- net N$44: now also R57.2, R58.1; no longer R56.2, R57.1
- net N$45: now also R56.2, R57.1; no longer R55.2, R56.1
- net N$5: now also RN15A.2, RN15B.1; no longer RN14A.2, RN14B.1
- net N$50: now also R36.2; no longer R31.2
- net N$53: now also R26.2, R28.2; no longer R21.2, R23.2
- net N$56: now also R39.2; no longer R34.2
- net N$58: now also R20.2, R22.2; no longer R15.2, R17.2
- net N$6: now also R15.1; no longer R9.1
- net N$62: now also R37.1, R38.2; no longer R32.1, R33.2
- net N$63: now also LED2.A, R2.1; no longer LED1.A, R11.1
- net N$68: now also R33.2; no longer R28.2
- net N$7: now also R58.2; no longer R57.2
- net NCE: now also R12.1; no longer R7.1
- net NCONFIG: now also R11.1; no longer R6.1
- net NSTATUS: now also R10.1; no longer R5.1
- net R: now also R42.2; no longer R37.2
- net SCK1: now also RN14A.2; no longer R40.2
- net SCK2: now also RN14B.1; no longer R42.2
- net SND: now also R44.1, R50.1; no longer R43.1, R49.1
- net SND4: now also R31.1; no longer R26.1
- net SND5: now also R30.1; no longer R25.1
- net SND_DAC: now also R29.1, R30.2, R32.2; no longer R24.1, R25.2, R27.2
- net SND_EXT: now also R48.1; no longer R45.1
- net TCK: now also R13.1; no longer R8.1
- net TDI: now also R7.1; no longer R2.1
- net TMS: now also R8.1; no longer R3.1
- net VCC: now also R2.2, R54.1, RN15B.2, RN15C.2; no longer R11.2, R53.1, RN14B.2, RN14C.2
- net VCCIO: now also D3.A, R10.2, R11.2, R17.1, R18.1, R19.1, R5.1, R6.1, R7.2, R8.2, R9.1; no longer R12.1, R13.1, R14.1, R2.2, R3.2, R5.2, R59.1, R6.2, R60.1, R62.1, X1-4.S
- net VPPL3: now also R51.1, R54.2, R56.1; no longer R50.1, R53.2, R54.1
Other:
- note added: "POWER ON"
- moved on the sheet: LED1, LED2, R1, R10, R11, R12, R13, R14, R15, R16, R17, R18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
